File: BTS7960.kicad_sch (KiCad schematic)
At the start: 4 parts, among them J2 Driver_2, J3 Driver_1, J4 Driver_3, J5 Driver_4

Commit message: Revision 110625
Parts:
- J2, J3, J4, J5: footprint (none) -> Connector_Molex:Molex_Micro-Fit_3.0_43045-0600_2x03_P3.00mm_Horizontal
Connections:
- net 5V renamed +5V
