File: I2C.kicad_sch (KiCad schematic)
At the start: 15 parts, among them J10 Sensor_2_right, J11 Sensor_3_left, J12 Sensor_4_back, J14 Sensor_1_front, U2 ICM-20948, U5 TCA9548APWR

Commit message: Revision 110625
Parts:
- removed J10: Sensor_2_right, symbol Connector:Conn_01x05_Socket
- removed J11: Sensor_3_left, symbol Connector:Conn_01x05_Socket
- removed J12: Sensor_4_back, symbol Connector:Conn_01x05_Socket
- removed J14: Sensor_1_front, symbol Connector:Conn_01x05_Socket
- added J10: Sproximidad_2, Connector_Molex:Molex_Micro-Fit_3.0_43045-0400_2x02_P3.00mm_Horizontal, symbol Connector:Conn_01x04_Socket
- added J11: Sproximidad_3, Connector_Molex:Molex_Micro-Fit_3.0_43045-0400_2x02_P3.00mm_Horizontal, symbol Connector:Conn_01x04_Socket
- added J12: Sproximidad_4, Connector_Molex:Molex_Micro-Fit_3.0_43045-0400_2x02_P3.00mm_Horizontal, symbol Connector:Conn_01x04_Socket
- added J14: Sproximidad_1, Connector_Molex:Molex_Micro-Fit_3.0_43045-0400_2x02_P3.00mm_Horizontal, symbol Connector:Conn_01x04_Socket
- C5: value 0.1uF -> 100nF; footprint Capacitor_SMD:C_0201_0603Metric -> Capacitor_SMD:C_0805_2012Metric; LCSC Part # (none) -> C49678
- C6, C7, C8: value 0.1uF -> 100nF; footprint (none) -> Capacitor_SMD:C_0805_2012Metric; LCSC Part # (none) -> C49678
- R1, R2, R4, R5: footprint (none) -> Resistor_SMD:R_0805_2012Metric; LCSC Part # (none) -> C17673
- R3: footprint (none) -> Resistor_SMD:R_0805_2012Metric; LCSC Part # (none) -> C17414
- U2: LCSC Part # (none) -> C726001
- U5: LCSC Part # (none) -> C130026
Connections:
- net GND: now also J10.2 (Pin_2), J11.2 (Pin_2), J12.2 (Pin_2), J14.2 (Pin_2)
- net at U5.11 (SC3): now also J12.3 (Pin_3)
- net at U5.10 (SD3): now also J12.4 (Pin_4)
- net at U5.4 (SD0): now also J14.4 (Pin_4)
- net at U5.5 (SC0): now also J14.3 (Pin_3)
- net at U5.6 (SD1): now also J10.4 (Pin_4)
- net at U5.7 (SC1): now also J10.3 (Pin_3)
- net at U5.8 (SD2): now also J11.4 (Pin_4)
- net at U5.9 (SC2): now also J11.3 (Pin_3)
- net 3.3V renamed +3V3
- net +3V3: now also J10.1 (Pin_1), J11.1 (Pin_1), J12.1 (Pin_1), J14.1 (Pin_1)
- net PB10 renamed PB8
- net PB11 renamed PB9
