File: Microcontrolador.kicad_sch (KiCad schematic)
At the start: 24 parts, among them J15 Conn_01x05_Socket, Q1 S8050, SW1 SW_Push, SW2 SW_Push, U3 STM32F407VGTx

Commit message: Revision 110625
Parts:
- removed BZ1: Buzzer, Buzzer_Beeper:Buzzer_D14mm_H7mm_P10mm, symbol Device:Buzzer
- removed Q1: S8050, Package_TO_SOT_THT:TO-92_Inline, symbol Transistor_BJT:S8050
- added C20: 1uF, Capacitor_SMD:C_0805_2012Metric, symbol Device:C
- added LS1: CMT-8540S-SMT, CUI_CMT-8540S-SMT, symbol CMT-8540S-SMT:CMT-8540S-SMT
- added Q1: SS8050, Package_TO_SOT_SMD:SOT-23, symbol Transistor_BJT:SS8050
- added R37: 100ohm, Resistor_SMD:R_0805_2012Metric, symbol Device:R
- C1, C13, C14, C15, C16, C18, C19, C2, C9: footprint Capacitor_SMD:C_0201_0603Metric -> Capacitor_SMD:C_0805_2012Metric; LCSC Part # (none) -> C49678
- C17: footprint Capacitor_SMD:C_0201_0603Metric -> Capacitor_SMD:C_0805_2012Metric; LCSC Part # (none) -> C28323
- C3, C4: footprint Capacitor_SMD:C_0201_0603Metric -> Capacitor_SMD:C_0805_2012Metric
- D4: footprint Diode_THT:D_DO-35_SOD27_P7.62mm_Horizontal -> Diode_SMD:D_SOD-323F; LCSC Part # (none) -> C2128
- FB2: value 100-220 Ω @100 MHz -> 600 Ω a 100 MHz; footprint (none) -> Inductor_SMD:L_0603_1608Metric; LCSC Part # (none) -> C141723
- J15: footprint (none) -> Connector_PinHeader_2.54mm:PinHeader_1x05_P2.54mm_Vertical
- R12, R36, R6: value 10k -> 10kohm; footprint Resistor_SMD:R_0201_0603Metric -> Resistor_SMD:R_0805_2012Metric; LCSC Part # (none) -> C17414
- R29: footprint Resistor_SMD:R_0201_0603Metric -> Resistor_SMD:R_0805_2012Metric; LCSC Part # (none) -> C17513
- SW1, SW2: footprint Button_Switch_SMD:SW_SPST_PTS645 -> Button_Switch_SMD:SW_SPST_TL3342; LCSC Part # (none) -> C318884
- U3: LCSC Part # (none) -> C12345
Connections:
- net GND: now also C20.1, Q1.2 (E); no longer U3.94 (BOOT0)
- net PA6: no longer R29.1
- net BOOT0: now reaches R12.2, SW2.1
- net BOOT0: now also U3.94 (BOOT0)
- net at D4.2 (A): now also LS1.N, Q1.3 (C)
- net at R29.2: now also Q1.1 (B)
- net BOOT1: now reaches R36.1, U3.37 (PB2)
- net PE2: now reaches U3.1 (PE2)
- net PC0: now reaches U3.15 (PC0)
- net PC3: now reaches U3.18 (PC3)
- net PE3: now reaches U3.2 (PE3)
- net at U3.21 (VREF+): now also C20.2, R37.1
- net PA4: now reaches U3.29 (PA4)
- net PE4: now reaches U3.3 (PE4)
- net PA5: now reaches U3.30 (PA5)
- net PC4: now reaches U3.33 (PC4)
- net PC5: now reaches U3.34 (PC5)
- net PB0: now reaches U3.35 (PB0)
- net PB1: now reaches U3.36 (PB1)
- net PE7: now reaches U3.38 (PE7)
- net PE8: now reaches U3.39 (PE8)
- net PE5: now reaches U3.4 (PE5)
- net PE10: now reaches U3.41 (PE10)
- net PE12: now reaches U3.43 (PE12)
- net PE15: now reaches U3.46 (PE15)
- net PE6: now reaches U3.5 (PE6)
- net PD8: now reaches U3.55 (PD8)
- net PD9: now reaches U3.56 (PD9)
- net PD12: now reaches U3.59 (PD12)
- net PD13: now reaches U3.60 (PD13)
- net PD14: now reaches U3.61 (PD14)
- net PD15: now reaches U3.62 (PD15)
- net PC6: now reaches U3.63 (PC6)
- net PC6: now also R29.1
- net PC7: now reaches U3.64 (PC7)
- net PC8: now reaches U3.65 (PC8)
- net PC9: now reaches U3.66 (PC9)
- net PA10: now reaches U3.69 (PA10)
- net PC13: now reaches U3.7 (PC13)
- net PA11: now reaches U3.70 (PA11)
- net PA12: now reaches U3.71 (PA12)
- net PA15: now reaches U3.77 (PA15)
- net PC10: now reaches U3.78 (PC10)
- net PC11: now reaches U3.79 (PC11)
- net PC14: now reaches U3.8 (PC14)
- net PC12: now reaches U3.80 (PC12)
- net PD0: now reaches U3.81 (PD0)
- net PD1: now reaches U3.82 (PD1)
- net PD2: now reaches U3.83 (PD2)
- net PD3: now reaches U3.84 (PD3)
- net PD4: now reaches U3.85 (PD4)
- net PD5: now reaches U3.86 (PD5)
- net PD6: now reaches U3.87 (PD6)
- net PD7: now reaches U3.88 (PD7)
- net PB3: now reaches U3.89 (PB3)
- net PC15: now reaches U3.9 (PC15)
- net PB4: now reaches U3.90 (PB4)
- net PB5: now reaches U3.91 (PB5)
- net PB8: now reaches U3.95 (PB8)
- net PB9: now reaches U3.96 (PB9)
- net PE0: now reaches U3.97 (PE0)
- net PE1: now reaches U3.98 (PE1)
- net 3.3V renamed +3V3
- net +3V3: now also R37.2
- net 5V renamed +5V
- net +5V: now also LS1.P
- no-connect marks 0 -> 2
Other:
- moved on the sheet: C3, C4, C9, D4, R12, R36, R6, SW1, SW2
