File: Placa_principal_v2.kicad_sch (KiCad schematic)
At the start: 0 parts

Commit message: Revision 110625
Other:
- added sheet Test_points (Test_points.kicad_sch)
Changed lines of the file:
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@@
+	)
+	(sheet
+		(at 189.23 128.27)
+		(size 43.18 20.32)
+		(fields_autoplaced yes)
+		(stroke
+			(width 0.1524)
+			(type solid)
+		)
+		(fill
+			(color 0 0 0 0.0000)
+		)
+		(property "Sheetname" "Test_points"
+			(at 189.23 127.5584 0)
+			(effects
+				(font
+					(size 1.27 1.27)
+				)
+				(justify left bottom)
+			)
+		)
+		(property "Sheetfile" "Test_points.kicad_sch"
+			(at 189.23 149.1746 0)
+			(effects
+				(font
+					(size 1.27 1.27)
+				)
+				(justify left top)
+			)
+		)
+		(instances
+			(project "Placa_principal_v2"
+				(path "/b0e8f483-0023-4ae8-ade5-8b5c3c2eccb2"
+					(page "9")
+				)
+			)
+		)
 	)
 	(sheet
