File: UART.kicad_sch (KiCad schematic)
At the start: 17 parts, among them J13 Conn_01x06_Socket, P1 USB_C_Plug_USB2.0, P2 USB_C_Plug_USB2.0, Q2 IRLML6402, U6 USBLC6-2SC6, U7 USBLC6-2SC6, U8 CH340G

Commit message: Revision 110625
Parts:
- removed D1, D3: D_Schottky, symbol Device:D_Schottky
- removed P1: USB_C_Plug_USB2.0, symbol Connector:USB_C_Plug_USB2.0
- removed P2: USB_C_Plug_USB2.0, Connector_USB:USB_C_Receptacle_GCT_USB4135-GF-A_6P_TopMnt_Horizontal, symbol Connector:USB_C_Plug_USB2.0
- added D1, D3: BAT54C, Package_TO_SOT_SMD:SOT-23, symbol Diode:BAT54C
- added D6: LED, LED_SMD:LED_0805_2012Metric, symbol Device:LED
- added J18, J19: USB_C_Receptacle_USB2.0_16P, Connector_USB:USB_C_Receptacle_GCT_USB4105-xx-A_16P_TopMnt_Horizontal, symbol Connector:USB_C_Receptacle_USB2.0_16P
- added R39: 270ohm, Resistor_SMD:R_0805_2012Metric, symbol Device:R
- C10: footprint Capacitor_SMD:C_0201_0603Metric -> Capacitor_SMD:C_0805_2012Metric; LCSC Part # (none) -> C49678
- J13: footprint (none) -> Connector_PinSocket_2.54mm:PinSocket_1x06_P2.54mm_Vertical
- Q2: LCSC Part # (none) -> C2593
- R10, R11, R31, R32, R9: footprint (none) -> Resistor_SMD:R_0805_2012Metric; LCSC Part # (none) -> C27834
- R7, R8: value 10k -> 10kohm; footprint (none) -> Resistor_SMD:R_0805_2012Metric; LCSC Part # (none) -> C17414
- U6, U7: LCSC Part # (none) -> C7519
- U8: LCSC Part # (none) -> C14267
Connections:
- net GND: now also R8.2, D6.1 (K), J18.A1 (GND), J18.A12 (GND), J18.B1 (GND), J18.B12 (GND), J18.S1 (SHIELD), J19.A1 (GND), J19.A12 (GND), J19.B1 (GND), J19.B12 (GND), J19.S1 (SHIELD); no longer R8.1
- net PA9: now also R8.1; no longer R8.2
- net PA9': now also D1.3, D3.3
- net at R10.2: now also J19.A5 (CC1)
- net USB1_D-: now reaches U6.4 (I/O2)
- net USB1_D-: now also J19.A7 (D-), J19.B7 (D-)
- net at U6.5 (VBUS): now also D3.1, J19.A4 (VBUS), J19.A9 (VBUS), J19.B4 (VBUS), J19.B9 (VBUS)
- net USB1_D+: now reaches U6.6 (I/O1)
- net USB1_D+: now also J19.A6 (D+), J19.B6 (D+)
- net at R11.2: now also J19.B5 (CC2)
- net at R32.2: now also J18.A5 (CC1)
- net UD+: now reaches U7.1 (I/O1), U8.5 (UD+)
- net UD+: no longer U7.5 (VBUS)
- net UD-: now reaches U7.3 (I/O2), U8.6 (UD-)
- net USB2_D-: now reaches U7.4 (I/O2)
- net USB2_D-: now also J18.A7 (D-), J18.B7 (D-)
- net USB2_D+: now reaches U7.6 (I/O1)
- net USB2_D+: now also J18.A6 (D+), J18.B6 (D+)
- net at R31.2: now also J18.B5 (CC2)
- net 3.3V renamed +3V3
- net +3V3: now also R39.2
- new net: D6.2 (A), R39.1
- new net VBUS_USB_2: D1.1, J18.A4 (VBUS), J18.A9 (VBUS), J18.B4 (VBUS), J18.B9 (VBUS), U7.5 (VBUS)
- no-connect marks 11 -> 17
Other:
- moved on the sheet: R8, R9
