File: _autosave-Placa_principal_v2.kicad_pcb (KiCad board)
At the start: 2 copper layers, 142.9 x 100.2 mm, 122 parts, among them J1 Encoder_1, J10 Sproximidad_2, J11 Sproximidad_3, J12 Sproximidad_4, J13 Conn_01x06_Socket, J14 Sproximidad_1, J15 Conn_01x05_Socket, J16 S_linea1, J17 S_linea2, J18 USB_C_Receptacle_USB2.0_16P, J19 USB_C_Receptacle_USB2.0_16P, J2 Driver_2, J20 Conn_02x10_Top_Bottom, J3 Driver_1, J4 Driver_3, J5 Driver_4, J6 Input 12V-24V connector, J7 Encoder_3, J8 Encoder_2, J9 Encoder_4, Q1 SS8050, Q2 IRLML6402, SW1 SW_Push, SW2 SW_Push, U1 LM1117MP-3.3, U2 ICM-20948, U3 STM32F407VGTx, U4 LM2596S-5, U5 TCA9548APWR, U6 USBLC6-2SC6, U7 USBLC6-2SC6, U8 CH340G

Commit message: Revision 110625
Parts:
- moved C7 11.7 mm to (194.9, 99.0), turned to 0 degrees
- moved C6 8.34 mm to (188.7, 108.8), turned to 180 degrees
- turned C5 to 0 degrees
Routing:
- net Net-(U2-REGOUT): track 3.35 -> 5.17 mm
