File: sensoresdelinea.kicad_sch (KiCad schematic)
At the start: 6 parts, among them J16 Conn_01x03_Socket, J17 Conn_01x03_Socket

Commit message: Revision 110625
Parts:
- added J20: Conn_02x10_Top_Bottom, Connector_PinSocket_2.54mm:PinSocket_2x10_P2.54mm_Vertical, symbol Connector_Generic:Conn_02x10_Top_Bottom
- J16: value Conn_01x03_Socket -> S_linea1; footprint (none) -> Connector_Molex:Molex_Micro-Fit_3.0_43650-0300_1x03_P3.00mm_Horizontal
- J17: value Conn_01x03_Socket -> S_linea2; footprint (none) -> Connector_Molex:Molex_Micro-Fit_3.0_43650-0300_1x03_P3.00mm_Horizontal
- R30, R34: value 10k -> 10kohm; footprint (none) -> Resistor_SMD:R_0805_2012Metric; LCSC Part # (none) -> C17414
- R33, R35: footprint (none) -> Resistor_SMD:R_0805_2012Metric; LCSC Part # (none) -> C27834
Connections:
- net GND: now also J20.10 (Pin_10), J20.11 (Pin_11)
- net 5V renamed +5V
- net +5V: now also J20.20 (Pin_20)
- net PE9 renamed PE7
- new net +3V3: J20.1 (Pin_1)
- new net PA10: J20.4 (Pin_4)
- new net PA15: J20.5 (Pin_5)
- new net PA7: J20.2 (Pin_2)
- new net PA8: J20.3 (Pin_3)
- new net PB0: J20.6 (Pin_6)
- new net PB1: J20.7 (Pin_7)
- new net PB3: J20.8 (Pin_8)
- new net PB4: J20.9 (Pin_9)
- new net PB5: J20.12 (Pin_12)
- new net PC0: J20.13 (Pin_13)
- new net PC11: J20.16 (Pin_16)
- new net PC3: J20.14 (Pin_14)
- new net PC9: J20.15 (Pin_15)
- no-connect marks 0 -> 3
